Commit message: use arm_id as namespace; extract cartesian impedance parameters to yaml; try adding dual arm cartesian with simple dual launch but fail with communication_constraints_violation

File: franka_description/robots/panda_arm.ros2_control.xacro (robot description, xacro)
@@ -1,5 +1,5 @@
 <?xml version="1.0"?>
 <robot xmlns:xacro="http://www.ros.org/wiki/xacro">
-  <xacro:macro name="panda_arm_ros2_control" params="ns robot_ip use_fake_hardware:=^|false fake_sensor_commands:=^|false">
+  <xacro:macro name="panda_arm_ros2_control" params="ns arm_id robot_ip use_fake_hardware:=^|false fake_sensor_commands:=^|false">
     <ros2_control name="FrankaHardwareInterface" type="system">
       <hardware>
@@ -11,4 +11,5 @@
         <xacro:unless value="${use_fake_hardware}">
           <plugin>franka_hardware/FrankaHardwareInterface</plugin>
+          <param name="arm_id">${arm_id}</param>
           <param name="robot_ip">${robot_ip}</param>
         </xacro:unless>

File: franka_description/robots/panda_arm.urdf.xacro (robot description, xacro)
@@ -13,4 +13,4 @@
   </xacro:if>
   <xacro:include filename="$(find franka_description)/robots/panda_arm.ros2_control.xacro"/>
-  <xacro:panda_arm_ros2_control ns="$(arg arm_id)" robot_ip="$(arg robot_ip)" use_fake_hardware="$(arg use_fake_hardware)" fake_sensor_commands="$(arg fake_sensor_commands)"/>
+  <xacro:panda_arm_ros2_control ns="$(arg arm_id)" arm_id="$(arg arm_id)" robot_ip="$(arg robot_ip)" use_fake_hardware="$(arg use_fake_hardware)" fake_sensor_commands="$(arg fake_sensor_commands)"/>
 </robot>
